File: malibotti.kicad_sch (KiCad schematic)
At the start: 23 parts, among them J1 Servos, J2 Servos & I2C, J3 I2C1, J4 I2C2, J5 I2C1, J6 I2C2, U1 ESP32-C3_SUPERMINI_SMD, U2 AS5600, U3 AS5600

Commit message: Improvements
Parts:
- removed D1: LED, liebler_OPTO:LED_1206_3216Metric_ReverseMount, symbol Device:LED
- removed R1: k1, Resistor_SMD:R_1206_3216Metric_Pad1.30x1.75mm_HandSolder, symbol Device:R
- added C3: u1, Capacitor_SMD:C_1206_3216Metric_Pad1.33x1.80mm_HandSolder, symbol Device:C
- added D21: RGB3, liebler_OPTO:SK6812MINI-E_REV, symbol liebler_OPTO:SK6812MINI-E_Reverse
- added J7: RGB, TestPoint:TestPoint_Pad_1.5x1.5mm, symbol Connector_Generic:Conn_01x01
- added J8: TX, TestPoint:TestPoint_Pad_1.5x1.5mm, symbol Connector_Generic:Conn_01x01
- added J9: RX, TestPoint:TestPoint_Pad_1.5x1.5mm, symbol Connector_Generic:Conn_01x01
- added SW8: BTN, liebler_MECH:SW_Push_1P1T_NO_6x6mm_H6.5mm_Reverse, symbol Switch:SW_Push
Connections:
- net +5V: now also C3.1, D21.1 (VDD)
- net GND: now also C3.2, D21.3 (GND), SW8.2
- net SCL1: now also U1.5 (GPIO5); no longer U1.7 (GPIO7)
- net SDA1: now also U1.6 (GPIO6); no longer U1.8 (GPIO8)
- net SRV1: now also U1.10 (GPIO10); no longer U1.20 (GPIO20)
- net SRV2: now also U1.7 (GPIO7); no longer U1.21 (GPIO21)
- net at U1.9 (GPIO9): now also SW8.1
- new net: D21.2 (DOUT), J7.1 (Pin_1)
- new net RGB_LED: D21.4 (DIN), U1.8 (GPIO8)
- new net RX: J9.1 (Pin_1), U1.20 (GPIO20)
- new net TX: J8.1 (Pin_1), U1.21 (GPIO21)
