File: pcb_v1/malibotti.kicad_pcb (KiCad board)
At the start: 2 copper layers, 100 x 55 mm, 30 parts, among them J1 Servos, J2 Servos & I2C, J3 I2C1, J4 I2C2, J5 I2C1, J6 I2C2, J7 RGB, J8 TX, J9 RX, SW8 BTN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

Commit message: moved files
Parts:
- removed J7: RGB, TestPoint:TestPoint_Pad_1.5x1.5mm
- removed J8: TX, TestPoint:TestPoint_Pad_1.5x1.5mm
- removed J9: RX, TestPoint:TestPoint_Pad_1.5x1.5mm
- D21: moved to F.Cu
- turned D21 to 0 degrees
Connections:
- D21 pad 2: Net-(D21-DOUT) -> unconnected-(D21-DOUT-Pad2)
- U1 pad 20: /RX -> unconnected-(U1-GPIO20-Pad20)
- U1 pad 21: /TX -> unconnected-(U1-GPIO21-Pad21)
Routing:
- net /RX: track 3.50 -> 0.00 mm
- net /TX: track 3.50 -> 0.00 mm
- net Net-(D21-DOUT): track 1.29 -> 0.00 mm
