File: pcb_v1/malibotti.kicad_sch (KiCad schematic)
At the start: 27 parts, among them J1 Servos, J2 Servos & I2C, J3 I2C1, J4 I2C2, J5 I2C1, J6 I2C2, J7 RGB, J8 TX, J9 RX, SW8 BTN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

Commit message: moved files
Parts:
- removed J7: RGB, TestPoint:TestPoint_Pad_1.5x1.5mm, symbol Connector_Generic:Conn_01x01
- removed J8: TX, TestPoint:TestPoint_Pad_1.5x1.5mm, symbol Connector_Generic:Conn_01x01
- removed J9: RX, TestPoint:TestPoint_Pad_1.5x1.5mm, symbol Connector_Generic:Conn_01x01
Connections:
- net RX: no longer names the net of U1.20 (GPIO20)
- net TX: no longer names the net of U1.21 (GPIO21)
- no-connect marks 4 -> 7
