File: malibotti_pcb_v2/malibotti_pcb_v2.kicad_pcb (KiCad board)
At the start: 2 copper layers, 67.5 x 55 mm, 43 parts, among them J2 Servos & I2C, J3 Servo1, J4 Servo2, J5 USB_C_Receptacle_USB2.0_16P, J6 Conn_01x04, SW1 RST, SW8 BTN, U1 ESP32-C3-MINI-1, U2 XC6206PxxxMR, U5 MX116H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

Commit message: Added serial port
Routing:
- net BUZZER: track 44.0 -> 45.7 mm
- net /TX: track 41.9 -> 42.9 mm
- net GND: vias 106 -> 110
Changed lines of the file:
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@@
 	)
 	(via
+		(at 148.3 86.2)
+		(size 0.6)
+		(drill 0.3)
+		(layers "F.Cu" "B.Cu")
+		(free yes)
+		(net 1)
+	)
+	(via
 		(at 150.8 121.4)
 		(size 0.6)
@@
 	)
 	(via
+		(at 149.4 114.9)
+		(size 0.6)
+		(drill 0.3)
+		(layers "F.Cu" "B.Cu")
+		(free yes)
+		(net 1)
+	)
+	(via
 		(at 139 85.85)
 		(size 0.6)
@@
 	)
 	(via
+		(at 146.8 84.7)
+		(size 0.6)
+		(drill 0.3)
+		(layers "F.Cu" "B.Cu")
+		(free yes)
+		(net 1)
+	)
+	(via
 		(at 139.6 77.3)
 		(size 0.6)
@@
 	)
 	(via
+		(at 144.8 84)
+		(size 0.6)
+		(drill 0.3)
+		(layers "F.Cu" "B.Cu")
+		(free yes)
+		(net 1)
+	)
+	(via
 		(at 127.8 94.75)
 		(size 0.6)
@@
 	)
 	(segment
-		(start 148.892116 108.151)
-		(end 148.595558 107.854442)
+		(start 147.549 108.151)
+		(end 147.5 108.2)
 		(width 0.25)
 		(layer "F.Cu")
@@
 	)
 	(segment
-		(start 150.626 108.151)
-		(end 148.892116 108.151)
+		(start 151.2 108.325)
+		(end 151.026 108.151)
 		(width 0.25)
 		(layer "F.Cu")
@@
 	)
 	(segment
-		(start 150.825 108.35)
-		(end 150.626 108.151)
+		(start 151.026 108.151)
+		(end 147.549 108.151)
 		(width 0.25)
 		(layer "F.Cu")
@@
 	)
 	(via
-		(at 150.825 108.35)
+		(at 151.2 108.325)
 		(size 0.6)
 		(drill 0.3)
@@
 	)
 	(via
-		(at 148.595558 107.854442)
+		(at 147.5 108.2)
 		(size 0.6)
 		(drill 0.3)
@@
 	)
 	(segment
-		(start 147.55 116.6)
-		(end 149.16219 116.6)
+		(start 151.2 108.325)
+		(end 151.198 108.325)
 		(width 0.25)
 		(layer "B.Cu")
@@
 	)
 	(segment
-		(start 147.949 107.207884)
+		(start 147.949 106.329442)
 		(end 147.949 87.98681)
 		(width 0.25)
@@
 	)
 	(segment
-		(start 148.595558 107.854442)
-		(end 147.949 107.207884)
+		(start 147.5 106.778442)
+		(end 147.949 106.329442)
 		(width 0.25)
 		(layer "B.Cu")
@@
 	)
 	(segment
-		(start 145.26219 85.3)
-		(end 142.65 85.3)
+		(start 150.999 114.76319)
+		(end 149.16219 116.6)
 		(width 0.25)
 		(layer "B.Cu")
@@
 	)
 	(segment
-		(start 150.999 114.76319)
-		(end 150.999 108.524)
+		(start 145.26219 85.3)
+		(end 142.65 85.3)
 		(width 0.25)
 		(layer "B.Cu")
@@
 	)
 	(segment
-		(start 149.16219 116.6)
+		(start 150.999 108.524)
 		(end 150.999 114.76319)
 		(width 0.25)
@@
 	)
 	(segment
-		(start 150.999 108.524)
-		(end 150.825 108.35)
+		(start 147.949 87.98681)
+		(end 145.26219 85.3)
 		(width 0.25)
 		(layer "B.Cu")
@@
 	)
 	(segment
-		(start 147.949 87.98681)
-		(end 145.26219 85.3)
+		(start 149.16219 116.6)
+		(end 147.55 116.6)
 		(width 0.25)
 		(layer "B.Cu")
@@
 	)
 	(segment
+		(start 147.5 108.2)
+		(end 147.5 106.778442)
+		(width 0.25)
+		(layer "B.Cu")
+		(net 7)
+	)
+	(segment
+		(start 151.198 108.325)
+		(end 150.999 108.524)
+		(width 0.25)
+		(layer "B.Cu")
+		(net 7)
+	)
+	(segment
 		(start 142.425 110.26)
 		(end 140.975 108.81)
@@
 	)
 	(segment
-		(start 149.325 107.7)
-		(end 151.3 107.7)
+		(start 151.8 107.7)
+		(end 148.7 107.7)
 		(width 0.25)
 		(layer "F.Cu")
@@
 	)
 	(segment
-		(start 151.3 107.7)
-		(end 151.45 107.55)
+		(start 148.7 107.7)
+		(end 148.131163 107.131163)
 		(width 0.25)
 		(layer "F.Cu")
@@
 	)
 	(segment
-		(start 148.625 107)
-		(end 149.325 107.7)
+		(start 148.131163 107.131163)
+		(end 148.125 107.131163)
 		(width 0.25)
 		(layer "F.Cu")
@@
 	)
 	(via
-		(at 148.625 107)
+		(at 148.125 107.131163)
 		(size 0.6)
 		(drill 0.3)
@@
 	)
 	(via
-		(at 151.45 107.55)
+		(at 151.8 107.7)
 		(size 0.6)
 		(drill 0.3)
@@
 	)
 	(segment
-		(start 148.4 87.8)
-		(end 145.449 84.849)
+		(start 151.826 108.574)
+		(end 151.826 108.584298)
+		(width 0.25)
+		(layer "B.Cu")
+		(net 46)
+	)
+	(segment
+		(start 151.826 108.584298)
+		(end 151.459298 108.951)
 		(width 0.25)
 		(layer "B.Cu")
@@
 	)
 	(segment
-		(start 151.45 107.55)
+		(start 151.45 108.951)
 		(end 151.45 114.95)
 		(width 0.25)
@@
 	)
 	(segment
-		(start 145.449 84.849)
-		(end 143.35 84.849)
+		(start 148.125 107.131163)
+		(end 148.125 107.05)
 		(width 0.25)
 		(layer "B.Cu")
@@
 	)
 	(segment
-		(start 148.625 107)
+		(start 148.125 107.05)
 		(end 148.4 106.775)
 		(width 0.25)
@@
 	)
 	(segment
-		(start 148.4 106.775)
-		(end 148.4 87.8)
+		(start 143.35 84.849)
+		(end 143.35 83.9725)
 		(width 0.25)
 		(layer "B.Cu")
@@
 	)
 	(segment
+		(start 151.459298 108.951)
+		(end 151.45 108.951)
+		(width 0.25)
+		(layer "B.Cu")
+		(net 46)
+	)
+	(segment
+		(start 148.4 87.8)
+		(end 145.449 84.849)
+		(width 0.25)
+		(layer "B.Cu")
+		(net 46)
+	)
+	(segment
 		(start 151.45 114.95)
 		(end 149 117.4)
@@
 	)
 	(segment
-		(start 143.35 84.849)
-		(end 143.35 83.9725)
+		(start 151.9 107.8)
+		(end 151.9 108.5)
+		(width 0.25)
+		(layer "B.Cu")
+		(net 46)
+	)
+	(segment
+		(start 151.8 107.7)
+		(end 151.9 107.8)
+		(width 0.25)
+		(layer "B.Cu")
+		(net 46)
+	)
+	(segment
+		(start 148.4 106.775)
+		(end 148.4 87.8)
+		(width 0.25)
+		(layer "B.Cu")
+		(net 46)
+	)
+	(segment
+		(start 145.449 84.849)
+		(end 143.35 84.849)
+		(width 0.25)
+		(layer "B.Cu")
+		(net 46)
+	)
+	(segment
+		(start 151.9 108.5)
+		(end 151.826 108.574)
 		(width 0.25)
 		(layer "B.Cu")

Commit message: Malibotti Stepper + renaming
Parts:
- moved R1 8.15 mm to (132.5, 77.1), turned to 90 degrees
- moved C2 6.88 mm to (135.2, 90.0), turned to 180 degrees
- moved C5 3.10 mm to (127.9, 100.7)
- moved C10 3.04 mm to (104.3, 101.3)
- moved C9 3.04 mm to (104.3, 94.6)
- moved C14 3.00 mm to (127.4, 101.9)
- moved U6 2.70 mm to (124.7, 101.9), turned to -90 degrees
- moved U5 2.53 mm to (124.7, 97.2)
- moved C15 2.43 mm to (127.9, 98.7)
- moved C13 2.42 mm to (127.4, 97.5)
- moved J3 2.40 mm to (110.0, 97.2)
- moved J4 2.40 mm to (110.0, 104.0)
- moved R9 2.28 mm to (148.1, 82.8)
- moved R7 2.28 mm to (148.1, 81.0)
- moved R8 2.28 mm to (148.1, 81.9)
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Routing:
- net GND: track 19.3 -> 60.4 mm, vias 110 -> 120
- net Net-(J5-CC1): track 1.81 -> 10.4 mm, vias 0 -> 2
- net SERVO2_ADC: track 36.7 -> 40.9 mm
- net /M2_1: track 18.9 -> 22.0 mm
- net SERVO1_ADC: track 43.0 -> 46.1 mm
- net Net-(U1-EN/CHIP_PU): track 90.1 -> 93.2 mm
- net Vdrive: track 31.1 -> 34.2 mm
- net +5V: track 98.4 -> 95.5 mm
- net /M1_1: track 22.0 -> 24.7 mm
- net SERVO2_B: track 6.66 -> 4.15 mm
- net /M1_2: track 23.8 -> 26.2 mm
- net Net-(J5-CC2): track 5.24 -> 7.56 mm
- net Net-(J5-D+-PadA6): track 9.31 -> 11.6 mm
- net Net-(J5-D--PadA7): track 10.3 -> 12.5 mm
- net SERVO2_A: track 7.07 -> 8.47 mm
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Other:
- outline, holes or cut-outs redrawn
