File: malibotti_stepper_pcb/malibotti_stepper_pcb.kicad_sch (KiCad schematic)
At the start: 42 parts, among them J1 Stepper 1, J5 USB_C_Receptacle_USB2.0_16P, J6 Conn_01x04, SW1 RST, SW8 BTN, U1 ESP32-C3-MINI-1, U2 XC6206PxxxMR, U3 STSPIN220

Commit message: Malibotti WIP
Parts:
- removed TP2: M1_1, TestPoint:TestPoint_Pad_1.5x1.5mm, symbol Connector:TestPoint
- added C13, C14: 1n, Capacitor_SMD:C_0402_1005Metric, symbol Device:C
- added C15: u1, Capacitor_SMD:C_0402_1005Metric, symbol Device:C
- added C16: 22n, Capacitor_SMD:C_0402_1005Metric, symbol Device:C
- added C17: 22u, Capacitor_SMD:C_0603_1608Metric, symbol Device:C
- added C18: 2u2, Capacitor_SMD:C_0603_1608Metric, symbol Device:C
- added J2: Stepper 1, liebler_CONN:JST_XH_5P_SMD, symbol Connector_Generic_MountingPin:Conn_01x05_MountingPin
- added J3: Servo, Connector_PinHeader_2.54mm:PinHeader_1x03_P2.54mm_Vertical, symbol Connector_Generic:Conn_01x03
- added J4: Conn_01x04, liebler_CONN:JST_XH_S4B-XH-A-1_1x04_P2.50mm_Horizontal_SmallerCourtyard, symbol Connector_Generic:Conn_01x04
- added R15, R16, R17, R18: 1k, Resistor_SMD:R_0402_1005Metric, symbol Device:R
- added R19, R22, R23: 10k, Resistor_SMD:R_0402_1005Metric, symbol Device:R
- added R20, R21: 1r0, Resistor_SMD:R_0805_2012Metric_Pad1.20x1.40mm_HandSolder, symbol Device:R
- added R24, R25: 5k1, Resistor_SMD:R_0402_1005Metric, symbol Device:R
- added U4: STSPIN220, Package_DFN_QFN:VQFN-16-1EP_3x3mm_P0.5mm_EP1.8x1.8mm, symbol Driver_Motor:STSPIN220
- C7: footprint Capacitor_SMD:C_0603_1608Metric -> Capacitor_SMD:C_0402_1005Metric
- J1: footprint liebler_CONN:JST_XH_B5B-XH-A_1x05_P2.50mm_Vertical_smaller -> liebler_CONN:JST_XH_5P_SMD; symbol Connector_Generic:Conn_01x05 -> Connector_Generic_MountingPin:Conn_01x05_MountingPin
- R5, R6: value r33 -> 1r0; footprint (none) -> Resistor_SMD:R_0805_2012Metric_Pad1.20x1.40mm_HandSolder
Connections:
- net PWM is gone; now on net GND: R12.1
- net +3V3: now also J4.3 (Pin_3), R15.2, R16.2, R24.1, R25.2
- net +5V: now also C17.1, C18.1, J3.2 (Pin_2), U4.6 (VS)
- net BUZZER: no longer J6.2 (Pin_2), U1.30 (GPIO20/U0RXD)
- net GND: now also J1.MP (MountPin), C13.2, C14.2, C15.2, C16.2, C17.2, C18.2, J2.MP (MountPin), J3.3 (Pin_3), J4.4 (Pin_4), R17.1, R19.1, R20.2, R21.2, U4.15 (MODE2), U4.16 (MODE1), U4.17 (EPAD), U4.7 (GND)
- net SCL: now also J4.1 (Pin_1)
- net SDA: now also J4.2 (Pin_2)
- net at C8.1, R12.2, U3.11 (REF): now also R22.2
- net M1_1: no longer names the net of U1.16 (GPIO10)
- net M1_2: no longer names the net of U1.18 (GPIO4/ADC1_CH4)
- net M1_2: no longer TP3.1
- net M2_1: no longer names the net of U1.13 (GPIO1/ADC1_CH1/XTAL_32K_N)
- net M2_2: no longer names the net of U1.12 (GPIO0/ADC1_CH0/XTAL_32K_P)
- net SERVO1_ADC renamed DIR2
- net DIR2: now also U4.1 (DIR)
- net SERVO2_ADC renamed STEP2
- net STEP2: now also U4.2 (STCK)
- new net: R21.1, U4.9 (SENSEB)
- new net: J6.2 (Pin_2), U1.30 (GPIO20/U0RXD)
- new net: R23.1, R25.1
- new net: C15.1, R17.2, R23.2, U4.11 (REF)
- new net: J2.1 (Pin_1), U4.3 (OUTA1)
- new net: J2.2 (Pin_2), U4.10 (OUTB1)
- new net: J2.3 (Pin_3), U4.5 (OUTA2)
- new net: J2.4 (Pin_4), U4.8 (OUTB2)
- new net: C14.1, R16.1, U4.13 (EN/FLT)
- new net: R18.2, R19.2, U4.12 (TOFF)
- new net: R22.1, R24.2
- new net: R20.1, U4.4 (SENSEA)
- new net: C16.1, R18.1
- new net RESET2: C13.1, R15.1, U4.14 (STBY/RESET)
- new net Servo1: J3.1 (Pin_1)
- no-connect marks 4 -> 5
Other:
- moved on the sheet: C9, R13

Commit message: WIP
Parts:
- J3: footprint Connector_PinHeader_2.54mm:PinHeader_1x03_P2.54mm_Vertical -> Connector_PinHeader_2.54mm:PinHeader_1x03_P2.54mm_Vertical_SMD_Pin1Left
Connections:
- net RESET1 is gone; now on net STEPPER_RESET: C9.1, R13.1, U3.14 (STBY/RESET)
- net RESET2 is gone; now on net STEPPER_RESET: C13.1, R15.1, U4.14 (STBY/RESET)
- net SRV3 is gone; now on net Servo1: U1.19 (GPIO5/ADC2_CH0)
- net BUZZER: now also U1.12 (GPIO0/ADC1_CH0/XTAL_32K_P)
- net DIR1: now also U1.18 (GPIO4/ADC1_CH4)
- net STEP1: now also U1.16 (GPIO10)
- net RX: now reaches J6.2 (Pin_2), U1.30 (GPIO20/U0RXD)
- net STEPPER_RESET: now reaches U1.13 (GPIO1/ADC1_CH1/XTAL_32K_N)
Changed lines of the file:
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@@
 		)
 	)
+	(label "RX"
+		(at 116.84 43.18 0)
+		(effects
+			(font
+				(size 1.27 1.27)
+			)
+			(justify left bottom)
+		)
+	)
 	(label "USBD-"
 		(at 77.47 121.92 0)
@@
 		)
 	)
-	(global_label "RESET2"
+	(global_label "STEPPER_RESET"
 		(shape input)
 		(at 308.61 142.24 180)
@@
 		)
 		(property "Intersheetrefs" "${INTERSHEET_REFS}"
-			(at 298.6702 142.24 0)
+			(at 290.627 142.24 0)
 			(effects
 				(font
@@
 		)
 	)
+	(global_label "STEPPER_RESET"
+		(shape output)
+		(at 36.83 43.18 180)
+		(fields_autoplaced yes)
+		(effects
+			(font
+				(size 1.27 1.27)
+			)
+			(justify right)
+		)
+		(property "Intersheetrefs" "${INTERSHEET_REFS}"
+			(at 18.847 43.18 0)
+			(effects
+				(font
+					(size 1.27 1.27)
+				)
+				(justify right)
+				(hide yes)
+			)
+		)
+	)
+	(global_label "DIR1"
+		(shape output)
+		(at 92.71 66.04 0)
+		(fields_autoplaced yes)
+		(effects
+			(font
+				(size 1.27 1.27)
+			)
+			(justify left)
+		)
+		(property "Intersheetrefs" "${INTERSHEET_REFS}"
+			(at 100.0495 66.04 0)
+			(effects
+				(font
+					(size 1.27 1.27)
+				)
+				(justify left)
+				(hide yes)
+			)
+		)
+	)
+	(global_label "STEP1"
+		(shape output)
+		(at 92.71 81.28 0)
+		(fields_autoplaced yes)
+		(effects
+			(font
+				(size 1.27 1.27)
+			)
+			(justify left)
+		)
+		(property "Intersheetrefs" "${INTERSHEET_REFS}"
+			(at 101.5008 81.28 0)
+			(effects
+				(font
+					(size 1.27 1.27)
+				)
+				(justify left)
+				(hide yes)
+			)
+		)
+	)
 	(global_label "DIR1"
 		(shape input)
@@
 	(global_label "BUZZER"
 		(shape output)
-		(at 134.62 57.15 0)
+		(at 36.83 40.64 180)
 		(fields_autoplaced yes)
 		(effects
@@
 				(size 1.27 1.27)
 			)
-			(justify left)
+			(justify right)
 		)
 		(property "Intersheetrefs" "${INTERSHEET_REFS}"
-			(at 145.0437 57.15 0)
+			(at 26.4063 40.64 0)
 			(effects
 				(font
 					(size 1.27 1.27)
 				)
-				(justify left)
+				(justify right)
 				(hide yes)
 			)
@@
 		)
 	)
+	(global_label "STEPPER_RESET"
+		(shape input)
+		(at 130.81 137.16 180)
+		(fields_autoplaced yes)
+		(effects
+			(font
+				(size 1.27 1.27)
+			)
+			(justify right)
+		)
+		(property "Intersheetrefs" "${INTERSHEET_REFS}"
+			(at 112.827 137.16 0)
+			(effects
+				(font
+					(size 1.27 1.27)
+				)
+				(justify right)
+				(hide yes)
+			)
+		)
+	)
 	(global_label "SCL"
 		(shape bidirectional)
@@
 		)
 	)
-	(global_label "SRV3"
+	(global_label "Servo1"
 		(shape output)
 		(at 92.71 68.58 0)
@@
 		)
 		(property "Intersheetrefs" "${INTERSHEET_REFS}"
-			(at 100.4728 68.58 0)
+			(at 102.1056 68.58 0)
 			(effects
 				(font
@@
 		)
 	)
-	(global_label "RESET1"
-		(shape input)
-		(at 130.81 137.16 180)
-		(fields_autoplaced yes)
-		(effects
-			(font
-				(size 1.27 1.27)
-			)
-			(justify right)
-		)
-		(property "Intersheetrefs" "${INTERSHEET_REFS}"
-			(at 120.8702 137.16 0)
-			(effects
-				(font
-					(size 1.27 1.27)
-				)
-				(justify right)
-				(hide yes)
-			)
-		)
-	)
 	(global_label "SDA"
 		(shape bidirectional)
@@
 			)
 		)
-		(property "Footprint" "Connector_PinHeader_2.54mm:PinHeader_1x03_P2.54mm_Vertical"
+		(property "Footprint" "Connector_PinHeader_2.54mm:PinHeader_1x03_P2.54mm_Vertical_SMD_Pin1Left"
 			(at 210.82 36.83 0)
 			(effects
@@
 					(size 1.27 1.27)
 				)
-				(hide yes)
 			)
 		)

Commit message: WIP
Connections:
- net +3.3V is gone; now on net +3V3: U1.3 (3V3)

Commit message: Limit Switch
Parts:
- added SW2: MicroSwitchLeft, liebler_MECH:Omron D2F Left Angled, symbol Switch:SW_SPDT_312
- added SW3: MicroSwitchRight, liebler_MECH:Omron D2F Right Angled, symbol Switch:SW_SPDT_312
Connections:
- net BUZZER: now also SW2.1 (B), SW3.1 (B)
- net GND: now also SW2.2 (C), SW3.2 (C)
- no-connect marks 5 -> 7
