File: malibotti_stepper_pcb/malibotti_stepper_pcb.kicad_sch (KiCad schematic)
At the start: 64 parts, among them J1 Stepper 1, J2 Stepper 1, J3 Servo, J4 Conn_01x04, J5 USB_C_Receptacle_USB2.0_16P, J6 Conn_01x04, SW1 RST, SW2 MicroSwitchLeft, SW3 MicroSwitchRight, SW8 BTN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

Commit message: Malibotti stepper as ordered @ JLCPCB
Parts:
- removed TP3: M1_2, TestPoint:TestPoint_Pad_1.5x1.5mm, symbol Connector:TestPoint
- added TP1: TestPoint, TestPoint:TestPoint_Loop_D1.80mm_Drill1.0mm_Beaded, symbol Connector:TestPoint
- C12, C17, C2, C5: footprint Capacitor_SMD:C_0603_1608Metric -> Capacitor_SMD:C_0805_2012Metric
Connections:
- net GND: now also J5.SH (SHIELD); no longer J5.S1 (SHIELD)
- net at C10.1, R14.1, U3.13 (EN/FLT): now also TP1.1
