File: malibotti_stepper_pcb/malibotti_stepper_pcb.kicad_sch (KiCad schematic)
At the start: 64 parts, among them J1 Stepper 1, J2 Stepper 1, J3 Servo, J4 Conn_01x04, J5 USB_C_Receptacle_USB2.0_16P, J6 Conn_01x04, SW1 RST, SW2 MicroSwitchLeft, SW3 MicroSwitchRight, SW8 BTN, U1 ESP32-C3-MINI-1, U2 XC6206PxxxMR, U3 STSPIN220, U4 STSPIN220

Commit message: Malibotti unipolar as ordered @ JLCPCB
Parts:
- added R26: 10k, Resistor_SMD:R_0402_1005Metric, symbol Device:R
- J2: value Stepper 1 -> Stepper 2
- J4: value Conn_01x04 -> I2C
- TP1: footprint TestPoint:TestPoint_Loop_D1.80mm_Drill1.0mm_Beaded -> TestPoint:TestPoint_THTPad_D1.5mm_Drill0.7mm
Connections:
- net +3V3: now also R26.2
- net at SW1.1, U1.8 (EN/CHIP_PU): now also R26.1
Other:
- note added: "Mechanical"
- note added: "PSU"
- note added: "Stepper 1"
- note added: "Stepper 2"
- note added: "USB"
- moved on the sheet: BZ1, C1, C10, C11, C12, C13, C14, C15, C16, C17, C18, C2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
