File: malibotti_stepper_pcb/malibotti_stepper_pcb.kicad_sch (KiCad schematic)
At the start: 64 parts, among them J1 Stepper 1, J2 Stepper 1, J3 Servo, J4 Conn_01x04, J5 USB_C_Receptacle_USB2.0_16P, J6 Conn_01x04, SW1 RST, SW2 MicroSwitchLeft, SW3 MicroSwitchRight, SW8 BTN, U1 ESP32-C3-MINI-1, U2 XC6206PxxxMR, U3 STSPIN220, U4 STSPIN220

Commit message: Test mit Arduino-Stepper
Parts:
- added JP1: SolderJumper_3_Bridged12, Jumper:SolderJumper-3_P1.3mm_Bridged2Bar12_RoundedPad1.0x1.5mm_NumberLabels, symbol Jumper:SolderJumper_3_Bridged12
- added SW4: SW_Push, Button_Switch_THT:SW_PUSH_6mm_H13mm, symbol Switch:SW_Push
Connections:
- new net I2C:SCL_SENSOR: JP1.2 (C)
- new net SCL_ESP1: JP1.3 (B)
- new net SCL_ESP2: JP1.1 (A)
